File: hardware/HV_Carrier/12VBuck.kicad_sch (KiCad schematic)
At the start: 14 parts, among them U13 LMR51635XDDCR

Commit message: added bom
Parts:
- C89: LCSC P/N C6666325 -> C15849
- U13: P/N (none) -> LMR51635XDDCR
Changed lines of the file:
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@@
+			)
+		)
+		(property "P/N" "LMR51635XDDCR"
+			(at 114.3 81.28 0)
+			(hide yes)
+			(show_name no)
+			(do_not_autoplace no)
+			(effects
+				(font
+					(size 1.27 1.27)
+				)
 			)
 		)
@@
 			)
 		)
-		(property "LCSC P/N" "C6666325"
+		(property "LCSC P/N" "C15849"
 			(at 102.87 88.9 0)
 			(hide yes)
