File: hardware/HV_Carrier/AMC3311_OpAmp.kicad_sch (KiCad schematic)
At the start: 14 parts, among them U11 TLV9002QDRQ1

Commit message: added bom
Parts:
- C84: LCSC P/N (none) -> C14663
- R74, R75, R76, R77, R78, R79: LCSC P/N (none) -> C25804
Changed lines of the file:
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@@
+			)
+		)
+		(property "LCSC P/N" "C25804"
+			(at 86.36 113.03 90)
+			(hide yes)
+			(show_name no)
+			(do_not_autoplace no)
+			(effects
+				(font
+					(size 1.27 1.27)
+				)
 			)
 		)
@@
 			)
 		)
+		(property "LCSC P/N" "C25804"
+			(at 67.31 105.41 90)
+			(hide yes)
+			(show_name no)
+			(do_not_autoplace no)
+			(effects
+				(font
+					(size 1.27 1.27)
+				)
+			)
+		)
 		(pin "1"
 		)
@@
 		)
 		(property "P/N" "MLASH168SB7104KTNA01"
+			(at 170.18 86.36 0)
+			(hide yes)
+			(show_name no)
+			(do_not_autoplace no)
+			(effects
+				(font
+					(size 1.27 1.27)
+				)
+			)
+		)
+		(property "LCSC P/N" "C14663"
 			(at 170.18 86.36 0)
 			(hide yes)
@@
 			)
 		)
+		(property "LCSC P/N" "C25804"
+			(at 67.31 100.33 90)
+			(hide yes)
+			(show_name no)
+			(do_not_autoplace no)
+			(effects
+				(font
+					(size 1.27 1.27)
+				)
+			)
+		)
 		(pin "1"
 		)
@@
 			)
 		)
+		(property "LCSC P/N" "C25804"
+			(at 66.04 63.5 90)
+			(hide yes)
+			(show_name no)
+			(do_not_autoplace no)
+			(effects
+				(font
+					(size 1.27 1.27)
+				)
+			)
+		)
 		(pin "1"
 		)
@@
 			)
 		)
+		(property "LCSC P/N" "C25804"
+			(at 85.09 73.66 90)
+			(hide yes)
+			(show_name no)
+			(do_not_autoplace no)
+			(effects
+				(font
+					(size 1.27 1.27)
+				)
+			)
+		)
 		(pin "2"
 		)
@@
 			(at 66.04 68.58 90)
 			(hide yes)
+			(show_name no)
+			(do_not_autoplace no)
+			(effects
+				(font
+					(size 1.27 1.27)
+				)
+			)
+		)
+		(property "LCSC P/N" "C25804"
+			(at 66.04 68.58 90)
+			(hide yes)
