File: hardware/HV_Carrier/AMC3311_Sense.kicad_sch (KiCad schematic)
At the start: 17 parts, among them U4 AMC3311QDWERQ1

Commit message: added bom
Parts:
- C20, C21, C23, C25: LCSC P/N (none) -> C15849
Changed lines of the file:
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@@
+			)
+		)
+		(property "LCSC P/N" "C15849"
+			(at 198.12 71.12 0)
+			(hide yes)
+			(show_name no)
+			(do_not_autoplace no)
+			(effects
+				(font
+					(size 1.27 1.27)
+				)
 			)
 		)
@@
 			)
 		)
+		(property "LCSC P/N" "C15849"
+			(at 184.15 50.8 0)
+			(hide yes)
+			(show_name no)
+			(do_not_autoplace no)
+			(effects
+				(font
+					(size 1.27 1.27)
+				)
+			)
+		)
 		(pin "2"
 		)
@@
 		)
 		(property "P/N" "MLASH168SB7104KTNA01"
+			(at 99.06 57.15 90)
+			(hide yes)
+			(show_name no)
+			(do_not_autoplace no)
+			(effects
+				(font
+					(size 1.27 1.27)
+				)
+			)
+		)
+		(property "LCSC P/N" "C15849"
 			(at 99.06 57.15 90)
 			(hide yes)
@@
 			(at 99.06 64.77 90)
 			(hide yes)
+			(show_name no)
+			(do_not_autoplace no)
+			(effects
+				(font
+					(size 1.27 1.27)
+				)
+			)
+		)
+		(property "LCSC P/N" "C15849"
+			(at 99.06 64.77 90)
+			(hide yes)
