File: hardware/HV_Carrier/CAN_Transceiver.kicad_sch (KiCad schematic)
At the start: 9 parts, among them IC2 TCAN3413DR, U2 CDSOT23-T24CAN

Commit message: added bom
Parts:
- C13: LCSC P/N (none) -> C14663
Changed lines of the file:
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@@
+			)
+		)
+		(property "LCSC P/N" "C14663"
+			(at 189.23 88.9 0)
+			(hide yes)
+			(show_name no)
+			(do_not_autoplace no)
+			(effects
+				(font
+					(size 1.27 1.27)
+				)
 			)
 		)
