File: hardware/HV_Carrier/Current_Sense.kicad_sch (KiCad schematic)
At the start: 46 parts, among them J10 Shunt Conn, J11 SSA-2-100A, J12 Discharge Vin, J13 Charge Vin, J9 LZSR 80-P, U6 TLV9002QDRQ1

Commit message: added bom
Parts:
- C43, C44, C47, C48: LCSC P/N (none) -> C15849
- C50: LCSC P/N (none) -> C14663
- J10: P/N 1053091105 -> 1053091104
- J12, J13: P/N (none) -> 1053091102
- R35, R36, R37, R43, R44, R47: LCSC P/N (none) -> C25804
- R41, R42: P/N CR0603-JW-101ELF -> 0603WAF1000T5E
- R48: value 90k -> 90.9k; P/N (none) -> RMCF0603FT90K9
- R49: LCSC P/N (none) -> C25804; P/N (none) -> CRCW060310K0FKEI
Changed lines of the file:
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@@
 			)
 		)
+		(property "LCSC P/N" "C25804"
+			(at 77.47 60.96 90)
+			(hide yes)
+			(show_name no)
+			(do_not_autoplace no)
+			(effects
+				(font
+					(size 1.27 1.27)
+				)
+			)
+		)
 		(pin "1"
 		)
@@
 			)
 		)
+		(property "LCSC P/N" "C25804"
+			(at 171.45 46.99 90)
+			(hide yes)
+			(show_name no)
+			(do_not_autoplace no)
+			(effects
+				(font
+					(size 1.27 1.27)
+				)
+			)
+		)
 		(pin "2"
 		)
@@
 			)
 		)
+		(property "LCSC P/N" "C14663"
+			(at 245.11 38.1 0)
+			(hide yes)
+			(show_name no)
+			(do_not_autoplace no)
+			(effects
+				(font
+					(size 1.27 1.27)
+				)
+			)
+		)
 		(pin "2"
 		)
@@
 			)
 		)
-		(property "P/N" "CR0603-JW-101ELF"
+		(property "P/N" "0603WAF1000T5E"
 			(at 154.94 54.61 90)
 			(hide yes)
@@
 			)
 		)
+		(property "LCSC P/N" "C15849"
+			(at 52.07 40.64 90)
+			(hide yes)
+			(show_name no)
+			(do_not_autoplace no)
+			(effects
+				(font
+					(size 1.27 1.27)
+				)
+			)
+		)
 		(pin "1"
 		)
@@
 			)
 		)
-		(property "P/N" "1053091105"
+		(property "P/N" "1053091104"
 			(at 142.24 43.18 0)
 			(hide yes)
@@
 			)
 		)
+		(property "LCSC P/N" "C15849"
+			(at 52.07 30.48 90)
+			(hide yes)
+			(show_name no)
+			(do_not_autoplace no)
+			(effects
+				(font
+					(size 1.27 1.27)
+				)
+			)
+		)
 		(pin "1"
 		)
@@
 			)
 		)
+		(property "LCSC P/N" "C25804"
+			(at 171.45 54.61 90)
+			(hide yes)
+			(show_name no)
+			(do_not_autoplace no)
+			(effects
+				(font
+					(size 1.27 1.27)
+				)
+			)
+		)
 		(pin "2"
 		)
@@
 			)
 		)
+		(property "P/N" "1053091102"
+			(at 186.69 116.84 0)
+			(hide yes)
+			(show_name no)
+			(do_not_autoplace no)
+			(effects
+				(font
+					(size 1.27 1.27)
+				)
+			)
+		)
 		(pin "1"
 		)
@@
 			)
 		)
+		(property "LCSC P/N" "C25804"
+			(at 223.52 128.27 0)
+			(hide yes)
+			(show_name no)
+			(do_not_autoplace no)
+			(effects
+				(font
+					(size 1.27 1.27)
+				)
+			)
+		)
+		(property "P/N" "CRCW060310K0FKEI"
+			(at 223.52 128.27 0)
+			(hide yes)
+			(show_name no)
+			(do_not_autoplace no)
+			(effects
+				(font
+					(size 1.27 1.27)
+				)
+			)
+		)
 		(pin "1"
 		)
@@
 			)
 		)
+		(property "P/N" "1053091102"
+			(at 186.69 130.81 0)
+			(hide yes)
+			(show_name no)
+			(do_not_autoplace no)
+			(effects
+				(font
+					(size 1.27 1.27)
+				)
+			)
+		)
 		(pin "1"
 		)
@@
 			)
 		)
+		(property "LCSC P/N" "C15849"
+			(at 176.53 62.23 0)
+			(hide yes)
+			(show_name no)
+			(do_not_autoplace no)
+			(effects
+				(font
+					(size 1.27 1.27)
+				)
+			)
+		)
 		(pin "1"
 		)
@@
 			)
 		)
+		(property "LCSC P/N" "C25804"
+			(at 189.23 40.64 90)
+			(hide yes)
+			(show_name no)
+			(do_not_autoplace no)
+			(effects
+				(font
+					(size 1.27 1.27)
+				)
+			)
+		)
 		(pin "2"
 		)
@@
 			)
 		)
+		(property "LCSC P/N" "C15849"
+			(at 165.1 50.8 0)
+			(hide yes)
+			(show_name no)
+			(do_not_autoplace no)
+			(effects
+				(font
+					(size 1.27 1.27)
+				)
+			)
+		)
 		(pin "1"
 		)
@@
 			)
 		)
+		(property "LCSC P/N" "C25804"
+			(at 77.47 85.09 90)
+			(hide yes)
+			(show_name no)
+			(do_not_autoplace no)
+			(effects
+				(font
+					(size 1.27 1.27)
+				)
+			)
+		)
 		(pin "1"
 		)
@@
 			)
 		)
-		(property "Value" "90k"
+		(property "Value" "90.9k"
 			(at 226.06 115.5699 0)
 			(show_name no)
@@
 			)
 		)
+		(property "P/N" "RMCF0603FT90K9"
+			(at 223.52 114.3 0)
+			(hide yes)
+			(show_name no)
+			(do_not_autoplace no)
+			(effects
+				(font
+					(size 1.27 1.27)
+				)
+			)
+		)
 		(pin "1"
 		)
@@
 			)
 		)
-		(property "P/N" "CR0603-JW-101ELF"
+		(property "P/N" "0603WAF1000T5E"
 			(at 154.94 46.99 90)
 			(hide yes)
@@
 			(at 77.47 33.02 90)
 			(hide yes)
+			(show_name no)
+			(do_not_autoplace no)
+			(effects
+				(font
+					(size 1.27 1.27)
+				)
+			)
+		)
+		(property "LCSC P/N" "C25804"
+			(at 77.47 33.02 90)
+			(hide yes)
