File: hardware/HV_Carrier/Power_Mux.kicad_sch (KiCad schematic)
At the start: 8 parts, among them U10 TPS2117DRLR

Commit message: added bom
Parts:
- C78, C79, C80, C81: LCSC P/N (none) -> C14663
- R73: LCSC P/N (none) -> C25804
Changed lines of the file:
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@@
+			)
+		)
+		(property "LCSC P/N" "C14663"
+			(at 88.9 58.42 0)
+			(hide yes)
+			(show_name no)
+			(do_not_autoplace no)
+			(effects
+				(font
+					(size 1.27 1.27)
+				)
 			)
 		)
@@
 			)
 		)
+		(property "LCSC P/N" "C25804"
+			(at 76.2 68.58 0)
+			(hide yes)
+			(show_name no)
+			(do_not_autoplace no)
+			(effects
+				(font
+					(size 1.27 1.27)
+				)
+			)
+		)
 		(pin "1"
 		)
@@
 		)
 		(property "P/N" "MLASH168SB7104KTNA01"
+			(at 21.59 45.72 0)
+			(hide yes)
+			(show_name no)
+			(do_not_autoplace no)
+			(effects
+				(font
+					(size 1.27 1.27)
+				)
+			)
+		)
+		(property "LCSC P/N" "C14663"
 			(at 21.59 45.72 0)
 			(hide yes)
@@
 			)
 		)
+		(property "LCSC P/N" "C14663"
+			(at 40.64 68.58 0)
+			(hide yes)
+			(show_name no)
+			(do_not_autoplace no)
+			(effects
+				(font
+					(size 1.27 1.27)
+				)
+			)
+		)
 		(pin "1"
 		)
@@
 			(at 35.56 45.72 0)
 			(hide yes)
+			(show_name no)
+			(do_not_autoplace no)
+			(effects
+				(font
+					(size 1.27 1.27)
+				)
+			)
+		)
+		(property "LCSC P/N" "C14663"
+			(at 35.56 45.72 0)
+			(hide yes)
