File: hardware/HV_Carrier/USB-C Connector.kicad_sch (KiCad schematic)
At the start: 6 parts, among them J6 USB_C_Receptacle_USB2.0_16P

Commit message: added bom
Parts:
- J6: P/N (none) -> USB4105-GF-A-120
- R24, R25: P/N (none) -> 0603WAF5101T5E
Changed lines of the file:
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@@
+			)
+		)
+		(property "P/N" "0603WAF5101T5E"
+			(at 90.17 48.26 90)
+			(hide yes)
+			(show_name no)
+			(do_not_autoplace no)
+			(effects
+				(font
+					(size 1.27 1.27)
+				)
 			)
 		)
@@
 		)
 		(property "LCSC P/N" "C23186"
+			(at 97.79 48.26 90)
+			(hide yes)
+			(show_name no)
+			(do_not_autoplace no)
+			(effects
+				(font
+					(size 1.27 1.27)
+				)
+			)
+		)
+		(property "P/N" "0603WAF5101T5E"
 			(at 97.79 48.26 90)
 			(hide yes)
@@
 			(at 35.56 45.72 0)
 			(hide yes)
+			(show_name no)
+			(do_not_autoplace no)
+			(effects
+				(font
+					(size 1.27 1.27)
+				)
+			)
+		)
+		(property "P/N" "USB4105-GF-A-120"
+			(at 35.56 45.72 0)
+			(hide yes)
